Commit message: reworked

File: description/robot.urdf.xacro (robot description, xacro)
@@ -2,7 +2,8 @@
 <robot xmlns:xacro="http://www.ros.org/wiki/xacro"  name="robot">
     <xacro:arg name="sim_mode" default="true"/>
-    <xacro:include filename="youbot_base.xacro" />
+    <xacro:include filename="youbot_manip.xacro" />
+<!--
     <xacro:include filename="ros2_control.xacro" />
-    <xacro:include filename="lidar.xacro" />
+ -->
     <!-- <xacro:include filename="camera.xacro" /> -->
     <!-- <xacro:include filename="depth_camera.xacro" /> -->

File: description/ros2_control.xacro (robot description, xacro)
@@ -7,13 +7,5 @@
                 <param name="can">can0</param>
             </hardware>
-            <joint name="wheel_joint_fl">
-                <param name="node_id">2</param>
-                <param name="transmission">26</param>
-                <command_interface name="position"/>
-                <command_interface name="velocity"/>
-                <state_interface name="position"/>
-                <state_interface name="velocity"/>
-            </joint>
-            <joint name="wheel_joint_fr">
+            <joint name="arm_joint_1">
                 <param name="node_id">1</param>
                 <param name="transmission">26</param>
@@ -23,6 +15,6 @@
                 <state_interface name="velocity"/>
             </joint>
-            <joint name="wheel_joint_bl">
-                <param name="node_id">4</param>
+            <joint name="arm_joint_2">
+                <param name="node_id">12</param>
                 <param name="transmission">26</param>
                 <command_interface name="position"/>
@@ -31,6 +23,22 @@
                 <state_interface name="velocity"/>
             </joint>
-            <joint name="wheel_joint_br">
-                <param name="node_id">3</param>
+            <joint name="arm_joint_3">
+                <param name="node_id">13</param>
+                <param name="transmission">26</param>
+                <command_interface name="position"/>
+                <command_interface name="velocity"/>
+                <state_interface name="position"/>
+                <state_interface name="velocity"/>
+            </joint>
+            <joint name="arm_joint_4">
+                <param name="node_id">14</param>
+                <param name="transmission">26</param>
+                <command_interface name="position"/>
+                <command_interface name="velocity"/>
+                <state_interface name="position"/>
+                <state_interface name="velocity"/>
+            </joint>
+            <joint name="arm_joint_5">
+                <param name="node_id">15</param>
                 <param name="transmission">26</param>
                 <command_interface name="position"/>
@@ -74,6 +82,6 @@
     <gazebo>
         <plugin name="gz_ros2_control::GazeboSimROS2ControlPlugin" filename="libgz_ros2_control-system.so">
-            <parameters>$(find youbot)/config/controllers.yaml</parameters>
-            <parameters>$(find youbot)/config/gaz_ros2_ctl_use_sim.yaml</parameters>
+            <parameters>$(find manip)/config/controllers.yaml</parameters>
+            <parameters>$(find manip)/config/gaz_ros2_ctl_use_sim.yaml</parameters>
         </plugin>
     </gazebo>
@@ -81,5 +89,5 @@
         name="gz_ros2_control"
         filename="libgz_ros2_control-system.so">
-        <parameters>$(find youbot)/config/controllers.yaml</parameters>
+        <parameters>$(find manip)/config/controllers.yaml</parameters>
     </plugin> -->
 </robot>

File: description/youbot_all.xacro (robot description, xacro)
@@ -1,4 +1,4 @@
 <?xml version="1.0" ?>
-<robot name="youbot">
+<robot name="manip">
   <!-- Define materials -->
   <material name="black"><color rgba="0.0 0.0 0.0 1.0"/></material>
@@ -90,11 +90,11 @@
       <origin rpy="0 0 0" xyz="0 0 0"/>
       <geometry>
-        <mesh filename="file://$(find youbot)/meshes/youbot_base/base.dae"/>
-      </geometry>
-    </visual>
-    <collision>
-      <origin rpy="0 0 0" xyz="0 0 0"/>
-      <geometry>
-        <mesh filename="file://$(find youbot)/meshes/youbot_base/base_convex.dae"/>
+        <mesh filename="file://$(find manip)/meshes/manip_base/base.dae"/>
+      </geometry>
+    </visual>
+    <collision>
+      <origin rpy="0 0 0" xyz="0 0 0"/>
+      <geometry>
+        <mesh filename="file://$(find manip)/meshes/manip_base/base_convex.dae"/>
       </geometry>
     </collision>
@@ -131,5 +131,5 @@
       <origin rpy="0 0 0" xyz="0 0 0"/>
       <geometry>
-        <mesh filename="file://$(find youbot)/meshes/youbot_base/front-left_wheel.dae"/>
+        <mesh filename="file://$(find manip)/meshes/manip_base/front-left_wheel.dae"/>
       </geometry>
     </visual>
@@ -187,5 +187,5 @@
       <origin rpy="0 0 0" xyz="0 0 0"/>
       <geometry>
-        <mesh filename="file://$(find youbot)/meshes/youbot_base/front-right_wheel.dae"/>
+        <mesh filename="file://$(find manip)/meshes/manip_base/front-right_wheel.dae"/>
       </geometry>
     </visual>
@@ -244,5 +244,5 @@
       <origin rpy="0 0 0" xyz="0 0 0"/>
       <geometry>
-        <mesh filename="file://$(find youbot)/meshes/youbot_base/back-left_wheel.dae"/>
+        <mesh filename="file://$(find manip)/meshes/manip_base/back-left_wheel.dae"/>
       </geometry>
     </visual>
@@ -300,5 +300,5 @@
       <origin rpy="0 0 0" xyz="0 0 0"/>
       <geometry>
-        <mesh filename="file://$(find youbot)/meshes/youbot_base/back-right_wheel.dae"/>
+        <mesh filename="file://$(find manip)/meshes/manip_base/back-right_wheel.dae"/>
       </geometry>
     </visual>
@@ -340,5 +340,5 @@
       <origin rpy="0 0 0" xyz="0 0 0"/>
       <geometry>
-        <mesh filename="file://$(find youbot)/meshes/sensors/hokuyo.dae"/>
+        <mesh filename="file://$(find manip)/meshes/sensors/hokuyo.dae"/>
       </geometry>
       <material name="black"/>
@@ -347,5 +347,5 @@
       <origin rpy="0 0 0" xyz="0 0 0"/>
       <geometry>
-        <mesh filename="file://$(find youbot)/meshes/sensors/hokuyo_convex.dae"/>
+        <mesh filename="file://$(find manip)/meshes/sensors/hokuyo_convex.dae"/>
       </geometry>
     </collision>
@@ -443,5 +443,5 @@
       <origin rpy="0 0 0" xyz="0 0 -0.025"/>
       <geometry>
-        <mesh filename="file://$(find youbot)/meshes/youbot_plate/plate.dae"/>
+        <mesh filename="file://$(find manip)/meshes/manip_plate/plate.dae"/>
       </geometry>
     </visual>
@@ -449,5 +449,5 @@
       <origin rpy="0 0 0" xyz="0 0 -0.025"/>
       <geometry>
-        <mesh filename="file://$(find youbot)/meshes/youbot_plate/plate_convex.dae"/>
+        <mesh filename="file://$(find manip)/meshes/manip_plate/plate_convex.dae"/>
       </geometry>
     </collision>
@@ -472,5 +472,5 @@
       <origin rpy="0 0 0" xyz="0 0 0"/>
       <geometry>
-        <mesh filename="file://$(find youbot)/meshes/youbot_arm/arm0.dae"/>
+        <mesh filename="file://$(find manip)/meshes/manip_arm/arm0.dae"/>
       </geometry>
     </visual>
@@ -479,5 +479,5 @@
       <origin rpy="0 0 0" xyz="0 0 0"/>
       <geometry>
-        <mesh filename="file://$(find youbot)/meshes/youbot_arm/arm0_convex.dae"/>
+        <mesh filename="file://$(find manip)/meshes/manip_arm/arm0_convex.dae"/>
         <!--<cylinder length="0.078" radius="0.093"/>-->
       </geometry>
@@ -509,5 +509,5 @@
       <origin xyz="0 0 0" rpy="0 0 0" />
       <geometry>
-        <mesh filename="file://$(find youbot)/meshes/youbot_arm/arm1.dae"/>
+        <mesh filename="file://$(find manip)/meshes/manip_arm/arm1.dae"/>
       </geometry>
     </visual>
@@ -516,5 +516,5 @@
       <origin xyz="0 0 0.02" rpy="3.14159 0 0" />
       <geometry>
-        <mesh filename="file://$(find youbot)/meshes/youbot_arm/arm_joint_1_convex.stl"/>
+        <mesh filename="file://$(find manip)/meshes/manip_arm/arm_joint_1_convex.stl"/>
         <!--<cylinder length="0.102" radius="0.080"/>-->
       </geometry>
@@ -539,5 +539,5 @@
       <origin xyz="0.001 -0.03 0.077" rpy="0 0 0" />
       <geometry>
-        <mesh filename="file://$(find youbot)/meshes/youbot_arm/arm2.dae"/>
+        <mesh filename="file://$(find manip)/meshes/manip_arm/arm2.dae"/>
       </geometry>
     </visual>
@@ -546,5 +546,5 @@
       <origin rpy="-1.570795 -1.570795 0" xyz="0 0 0"/>
       <geometry>
-        <mesh filename="file://$(find youbot)/meshes/youbot_arm/arm_joint_2_convex.stl"/>
+        <mesh filename="file://$(find manip)/meshes/manip_arm/arm_joint_2_convex.stl"/>
         <!--<box size="0.074 0.082 0.222"/>-->
       </geometry>
@@ -568,5 +568,5 @@
       <origin rpy="0 0 0" xyz="0.000 0.027 0.08"/>
       <geometry>
-        <mesh filename="file://$(find youbot)/meshes/youbot_arm/arm3.dae"/>
+        <mesh filename="file://$(find manip)/meshes/manip_arm/arm3.dae"/>
       </geometry>
     </visual>
@@ -575,5 +575,5 @@
       <origin rpy="1.570795 0 3.14159" xyz="0 0 0"/>
       <geometry>
-        <mesh filename="file://$(find youbot)/meshes/youbot_arm/arm_joint_3_convex.stl"/>
+        <mesh filename="file://$(find manip)/meshes/manip_arm/arm_joint_3_convex.stl"/>
         <!--<box size="0.064 0.054 0.192"/>-->
       </geometry>
@@ -598,5 +598,5 @@
       <origin rpy="0 0 0" xyz="0 -0.008 0.026"/>
       <geometry>
-        <mesh filename="file://$(find youbot)/meshes/youbot_arm/arm4.dae"/>
+        <mesh filename="file://$(find manip)/meshes/manip_arm/arm4.dae"/>
       </geometry>
     </visual>
@@ -605,5 +605,5 @@
       <origin rpy="1.570795 0 3.14159" xyz="0 0 0"/>
       <geometry>
-        <mesh filename="file://$(find youbot)/meshes/youbot_arm/arm_joint_4_convex.stl"/>
+        <mesh filename="file://$(find manip)/meshes/manip_arm/arm_joint_4_convex.stl"/>
         <!--<box size="0.058 0.100 0.118"/>-->
       </geometry>
@@ -628,11 +628,11 @@
       <origin rpy="0 0 0" xyz="0 0 -0.019"/>
       <geometry>
-        <mesh filename="file://$(find youbot)/meshes/youbot_arm/arm5.dae"/>
-      </geometry>
-    </visual>
-    <collision>
-      <origin rpy="0 0 0" xyz="0 0 0"/>
-      <geometry>
-        <mesh filename="file://$(find youbot)/meshes/youbot_arm/arm_joint_5_convex.stl"/>
+        <mesh filename="file://$(find manip)/meshes/manip_arm/arm5.dae"/>
+      </geometry>
+    </visual>
+    <collision>
+      <origin rpy="0 0 0" xyz="0 0 0"/>
+      <geometry>
+        <mesh filename="file://$(find manip)/meshes/manip_arm/arm_joint_5_convex.stl"/>
         <!--<box size="0.054 0.096 0.030"/>-->
       </geometry>

File: your_robot.urdf (robot description, URDF)
Before this commit: robot youbot, 8 links, 7 joints
Links:
- link base_laser_front_link: geometry collision mesh filename=file:///home/nbf2/manip_ws/install/manip/share/manip/meshes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; visual mesh filename=file:///home/nbf2/manip_ws/install/manip/share/manip/meshes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
- link chassis: geometry collision mesh filename=file:///home/nbf2/manip_ws/install/manip/share/manip/meshes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; visual mesh filename=file:///home/nbf2/manip_ws/install/manip/share/manip/meshes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
- link wheel_link_bl: geometry collision cylinder length=0.05 radius=0.05; visual mesh filename=file:///home/nbf2/manip_ws/install/manip/share/manip/meshes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
- link wheel_link_br: geometry collision cylinder length=0.05 radius=0.05; visual mesh filename=file:///home/nbf2/manip_ws/install/manip/share/manip/meshes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
- link wheel_link_fl: geometry collision cylinder length=0.05 radius=0.05; visual mesh filename=file:///home/nbf2/manip_ws/install/manip/share/manip/meshes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
- link wheel_link_fr: geometry collision cylinder length=0.05 radius=0.05; visual mesh filename=file:///home/nbf2/manip_ws/install/manip/share/manip/meshes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
