Commit message: edit

File: description/youbot_manip.xacro (robot description, xacro)
@@ -80,5 +80,5 @@
     <!-- damping - N*s/m, N*s*m/rad -->
     <!-- friction - N, N*m -->
-    <limit effort="10000.0" lower="0" upper="5.89920788889" velocity="1.570795"/>
+    <!-- <limit effort="10000.0" lower="0" upper="5.89920788889" velocity="1.570795"/> -->
     <!--effort - N, N*m-->
     <!--velocity - m/s, rad/s-->
@@ -115,5 +115,5 @@
     <!--<calibration rising="${arm_2_ref}" falling="${arm_2_ref}"/>-->
     <dynamics damping="1" friction="1"/>
-    <limit effort="10000.0" lower="0" upper="2.70525805556" velocity="1.570795"/>
+    <!-- <limit effort="10000.0" lower="0" upper="2.70525805556" velocity="1.570795"/> -->
   </joint>
   <link name="arm_link_2">
@@ -144,5 +144,5 @@
     <axis xyz="0 1 0"/>
     <dynamics damping="1" friction="1"/>
-    <limit effort="10000.0" lower="-5.1836235" upper="0" velocity="1.570795"/>
+    <!-- <limit effort="10000.0" lower="-5.1836235" upper="0" velocity="1.570795"/> -->
   </joint>
   <link name="arm_link_3">
@@ -174,5 +174,5 @@
     <!--<calibration rising="${arm_4_ref}" falling="${arm_4_ref}"/>-->
     <dynamics damping="1" friction="1"/>
-    <limit effort="10000.0" lower="0" upper="3.57792194444" velocity="1.570795"/>
+    <!-- <limit effort="10000.0" lower="0" upper="3.57792194444" velocity="1.570795"/> -->
   </joint>
   <link name="arm_link_4">
@@ -204,5 +204,5 @@
     <!--<calibration rising="${arm_5_ref}" falling="${arm_5_ref}"/>-->
     <dynamics damping="1" friction="1"/>
-    <limit effort="10000.0" lower="0" upper="5.84684805556" velocity="1.570795"/>
+    <!-- <limit effort="10000.0" lower="0" upper="5.84684805556" velocity="1.570795"/> -->
   </joint>
   <link name="arm_link_5">
@@ -251,5 +251,5 @@
     <axis xyz="0 0 -1"/>
     <dynamics damping="1" friction="1"/>
-    <limit effort="10000.0" lower="0" upper="5.84684805556" velocity="1.570795"/>
+    <!-- <limit effort="10000.0" lower="0" upper="5.84684805556" velocity="1.570795"/> -->
   </joint>
   <gazebo reference="arm_link_0">

Commit message: edit

File: description/youbot_manip.xacro (robot description, xacro)
@@ -80,5 +80,5 @@
     <!-- damping - N*s/m, N*s*m/rad -->
     <!-- friction - N, N*m -->
-    <!-- <limit effort="10000.0" lower="0" upper="5.89920788889" velocity="1.570795"/> -->
+    <limit effort="10000.0" lower="0" upper="5.89920788889" velocity="1.570795"/>
     <!--effort - N, N*m-->
     <!--velocity - m/s, rad/s-->
@@ -115,5 +115,5 @@
     <!--<calibration rising="${arm_2_ref}" falling="${arm_2_ref}"/>-->
     <dynamics damping="1" friction="1"/>
-    <!-- <limit effort="10000.0" lower="0" upper="2.70525805556" velocity="1.570795"/> -->
+    <limit effort="10000.0" lower="0" upper="2.70525805556" velocity="1.570795"/>
   </joint>
   <link name="arm_link_2">
@@ -144,5 +144,5 @@
     <axis xyz="0 1 0"/>
     <dynamics damping="1" friction="1"/>
-    <!-- <limit effort="10000.0" lower="-5.1836235" upper="0" velocity="1.570795"/> -->
+    <limit effort="10000.0" lower="-5.1836235" upper="0" velocity="1.570795"/>
   </joint>
   <link name="arm_link_3">
@@ -174,5 +174,5 @@
     <!--<calibration rising="${arm_4_ref}" falling="${arm_4_ref}"/>-->
     <dynamics damping="1" friction="1"/>
-    <!-- <limit effort="10000.0" lower="0" upper="3.57792194444" velocity="1.570795"/> -->
+    <limit effort="10000.0" lower="0" upper="3.57792194444" velocity="1.570795"/>
   </joint>
   <link name="arm_link_4">
@@ -204,5 +204,5 @@
     <!--<calibration rising="${arm_5_ref}" falling="${arm_5_ref}"/>-->
     <dynamics damping="1" friction="1"/>
-    <!-- <limit effort="10000.0" lower="0" upper="5.84684805556" velocity="1.570795"/> -->
+    <limit effort="10000.0" lower="0" upper="5.84684805556" velocity="1.570795"/>
   </joint>
   <link name="arm_link_5">
@@ -251,5 +251,5 @@
     <axis xyz="0 0 -1"/>
     <dynamics damping="1" friction="1"/>
-    <!-- <limit effort="10000.0" lower="0" upper="5.84684805556" velocity="1.570795"/> -->
+    <limit effort="10000.0" lower="0" upper="5.84684805556" velocity="1.570795"/>
   </joint>
   <gazebo reference="arm_link_0">

Commit message: edit

File: description/youbot_manip.xacro (robot description, xacro)
@@ -80,5 +80,6 @@
     <!-- damping - N*s/m, N*s*m/rad -->
     <!-- friction - N, N*m -->
-    <limit effort="10000.0" lower="0" upper="5.89920788889" velocity="1.570795"/>
+    <!-- <limit effort="10000.0" lower="0" upper="5.89920788889" velocity="1.570795"/> -->
+    <limit effort="10000.0" lower="-0.5" upper="5.89920788889" velocity="1.570795"/>
     <!--effort - N, N*m-->
     <!--velocity - m/s, rad/s-->
@@ -115,5 +116,6 @@
     <!--<calibration rising="${arm_2_ref}" falling="${arm_2_ref}"/>-->
     <dynamics damping="1" friction="1"/>
-    <limit effort="10000.0" lower="0" upper="2.70525805556" velocity="1.570795"/>
+    <!-- <limit effort="10000.0" lower="0" upper="2.70525805556" velocity="1.570795"/> -->
+    <limit effort="10000.0" lower="-0.5" upper="2.70525805556" velocity="1.570795"/>
   </joint>
   <link name="arm_link_2">
@@ -144,5 +146,6 @@
     <axis xyz="0 1 0"/>
     <dynamics damping="1" friction="1"/>
-    <limit effort="10000.0" lower="-5.1836235" upper="0" velocity="1.570795"/>
+    <!-- <limit effort="10000.0" lower="-5.1836235" upper="0" velocity="1.570795"/> -->
+    <limit effort="10000.0" lower="-5.1836235" upper="0.5" velocity="1.570795"/>
   </joint>
   <link name="arm_link_3">
@@ -174,5 +177,6 @@
     <!--<calibration rising="${arm_4_ref}" falling="${arm_4_ref}"/>-->
     <dynamics damping="1" friction="1"/>
-    <limit effort="10000.0" lower="0" upper="3.57792194444" velocity="1.570795"/>
+    <!-- <limit effort="10000.0" lower="0" upper="3.57792194444" velocity="1.570795"/> -->
+    <limit effort="10000.0" lower="-0.5" upper="3.57792194444" velocity="1.570795"/>
   </joint>
   <link name="arm_link_4">
@@ -204,5 +208,6 @@
     <!--<calibration rising="${arm_5_ref}" falling="${arm_5_ref}"/>-->
     <dynamics damping="1" friction="1"/>
-    <limit effort="10000.0" lower="0" upper="5.84684805556" velocity="1.570795"/>
+    <!-- <limit effort="10000.0" lower="0" upper="5.84684805556" velocity="1.570795"/> -->
+    <limit effort="10000.0" lower="-0.5" upper="5.84684805556" velocity="1.570795"/>
   </joint>
   <link name="arm_link_5">
@@ -251,5 +256,6 @@
     <axis xyz="0 0 -1"/>
     <dynamics damping="1" friction="1"/>
-    <limit effort="10000.0" lower="0" upper="5.84684805556" velocity="1.570795"/>
+    <!-- <limit effort="10000.0" lower="0" upper="5.84684805556" velocity="1.570795"/> -->
+    <limit effort="10000.0" lower="-0.5" upper="5.84684805556" velocity="1.570795"/>
   </joint>
   <gazebo reference="arm_link_0">
