Commit message: Working PosContr

File: description/ros2_control.xacro (robot description, xacro)
@@ -5,5 +5,5 @@
             <hardware>
                 <plugin>odrive_ros2_control_plugin/ODriveHardwareInterface</plugin>
-                <param name="can">can1</param>
+                <param name="can">can0</param>
             </hardware>
             <joint name="arm_joint_1">

File: description/youbot_manip.xacro (robot description, xacro)
@@ -146,5 +146,5 @@
     <axis xyz="0 1 0"/>
     <dynamics damping="1" friction="1"/>
-    <limit effort="10000.0" lower="-5.1836235" upper="0" velocity="1.570795"/>
+    <limit effort="10000.0" lower="-5.1836235" upper="5" velocity="1.570795"/>
     <!-- <limit effort="10000.0" lower="-5.1836235" upper="0.5" velocity="1.570795"/> -->
   </joint>
@@ -288,5 +288,5 @@
     <actuator name="arm_motor_1">
       <hardwareInterface>EffortJointInterface</hardwareInterface>
-      <mechanicalReduction>1</mechanicalReduction>
+      <mechanicalReduction>156</mechanicalReduction>
     </actuator>
   </transmission>
@@ -296,5 +296,5 @@
     <actuator name="arm_motor_2">
       <hardwareInterface>EffortJointInterface</hardwareInterface>
-      <mechanicalReduction>1</mechanicalReduction>
+      <mechanicalReduction>156</mechanicalReduction>
     </actuator>
   </transmission>
@@ -304,5 +304,5 @@
     <actuator name="arm_motor_3">
       <hardwareInterface>EffortJointInterface</hardwareInterface>
-      <mechanicalReduction>1</mechanicalReduction>
+      <mechanicalReduction>71</mechanicalReduction>
     </actuator>
   </transmission>
@@ -312,5 +312,5 @@
     <actuator name="arm_motor_4">
       <hardwareInterface>EffortJointInterface</hardwareInterface>
-      <mechanicalReduction>1</mechanicalReduction>
+      <mechanicalReduction>100</mechanicalReduction>
     </actuator>
   </transmission>
@@ -320,5 +320,5 @@
     <actuator name="arm_motor_5">
       <hardwareInterface>EffortJointInterface</hardwareInterface>
-      <mechanicalReduction>1</mechanicalReduction>
+      <mechanicalReduction>100</mechanicalReduction>
     </actuator>
   </transmission>
