Commit message: working sim

File: build/manip/description/robot.urdf.xacro (robot description, xacro)
@@ -1 +1 @@
-/home/bfh/manip_ws/description/robot.urdf.xacro
+/home/nbf2/manip_ws/description/robot.urdf.xacro

File: build/manip/description/ros2_control.xacro (robot description, xacro)
@@ -1 +1 @@
-/home/bfh/manip_ws/description/ros2_control.xacro
+/home/nbf2/manip_ws/description/ros2_control.xacro

File: build/manip/description/youbot_all.xacro (robot description, xacro)
@@ -1 +1 @@
-/home/bfh/manip_ws/description/youbot_all.xacro
+/home/nbf2/manip_ws/description/youbot_all.xacro

File: build/manip/description/youbot_manip.xacro (robot description, xacro)
@@ -1 +1 @@
-/home/bfh/manip_ws/description/youbot_manip.xacro
+/home/nbf2/manip_ws/description/youbot_manip.xacro

File: description/ros2_control.xacro (robot description, xacro)
@@ -1,5 +1,5 @@
 <?xml version="1.0"?>
 <robot xmlns:xacro="http://www.ros.org/wiki/xacro">
-    <!-- <xacro:unless value="$(arg sim_mode)"> -->
+    <xacro:unless value="$(arg sim_mode)">
         <ros2_control name="RealRobot" type="system">
             <hardware>
@@ -48,5 +48,5 @@
             </joint>
         </ros2_control>
-    <!-- </xacro:unless>
+    </xacro:unless>
     <xacro:if value="$(arg sim_mode)">
         <ros2_control name="GazeboSystem" type="system">
@@ -54,5 +54,5 @@
                 <plugin>gz_ros2_control/GazeboSimSystem</plugin>
             </hardware>
-            <joint name="wheel_joint_fl">
+            <joint name="arm_joint_1">
                 <command_interface name="position"/>
                 <command_interface name="velocity"/>
@@ -60,5 +60,5 @@
                 <state_interface name="velocity"/>
             </joint>
-            <joint name="wheel_joint_fr">
+            <joint name="arm_joint_2">
                 <command_interface name="position"/>
                 <command_interface name="velocity"/>
@@ -66,5 +66,5 @@
                 <state_interface name="velocity"/>
             </joint>
-            <joint name="wheel_joint_bl">
+            <joint name="arm_joint_3">
                 <command_interface name="position"/>
                 <command_interface name="velocity"/>
@@ -72,5 +72,11 @@
                 <state_interface name="velocity"/>
             </joint>
-            <joint name="wheel_joint_br">
+            <joint name="arm_joint_4">
+                <command_interface name="position"/>
+                <command_interface name="velocity"/>
+                <state_interface name="position"/>
+                <state_interface name="velocity"/>
+            </joint>
+            <joint name="arm_joint_5">
                 <command_interface name="position"/>
                 <command_interface name="velocity"/>
@@ -85,9 +91,4 @@
             <parameters>$(find manip)/config/gaz_ros2_ctl_use_sim.yaml</parameters>
         </plugin>
-    </gazebo> -->
-    <!-- <plugin
-        name="gz_ros2_control"
-        filename="libgz_ros2_control-system.so">
-        <parameters>$(find manip)/config/controllers.yaml</parameters>
-    </plugin> -->
+    </gazebo>
 </robot>

File: description/youbot_manip.xacro (robot description, xacro)
@@ -80,6 +80,6 @@
     <!-- damping - N*s/m, N*s*m/rad -->
     <!-- friction - N, N*m -->
-    <!-- <limit effort="10000.0" lower="0" upper="5.89920788889" velocity="1.570795"/> -->
-    <limit effort="10000.0" lower="-0.5" upper="5.89920788889" velocity="1.570795"/>
+    <limit effort="10000.0" lower="0" upper="5.89920788889" velocity="1.570795"/>
+    <!-- <limit effort="10000.0" lower="-0.5" upper="5.89920788889" velocity="1.570795"/> -->
     <!--effort - N, N*m-->
     <!--velocity - m/s, rad/s-->
@@ -116,6 +116,6 @@
     <!--<calibration rising="${arm_2_ref}" falling="${arm_2_ref}"/>-->
     <dynamics damping="1" friction="1"/>
-    <!-- <limit effort="10000.0" lower="0" upper="2.70525805556" velocity="1.570795"/> -->
-    <limit effort="10000.0" lower="-0.5" upper="2.70525805556" velocity="1.570795"/>
+    <limit effort="10000.0" lower="0" upper="2.70525805556" velocity="1.570795"/>
+    <!-- <limit effort="10000.0" lower="-0.5" upper="2.70525805556" velocity="1.570795"/> -->
   </joint>
   <link name="arm_link_2">
@@ -146,6 +146,6 @@
     <axis xyz="0 1 0"/>
     <dynamics damping="1" friction="1"/>
-    <!-- <limit effort="10000.0" lower="-5.1836235" upper="0" velocity="1.570795"/> -->
-    <limit effort="10000.0" lower="-5.1836235" upper="0.5" velocity="1.570795"/>
+    <limit effort="10000.0" lower="-5.1836235" upper="0" velocity="1.570795"/>
+    <!-- <limit effort="10000.0" lower="-5.1836235" upper="0.5" velocity="1.570795"/> -->
   </joint>
   <link name="arm_link_3">
@@ -177,6 +177,6 @@
     <!--<calibration rising="${arm_4_ref}" falling="${arm_4_ref}"/>-->
     <dynamics damping="1" friction="1"/>
-    <!-- <limit effort="10000.0" lower="0" upper="3.57792194444" velocity="1.570795"/> -->
-    <limit effort="10000.0" lower="-0.5" upper="3.57792194444" velocity="1.570795"/>
+    <limit effort="10000.0" lower="0" upper="3.57792194444" velocity="1.570795"/>
+    <!-- <limit effort="10000.0" lower="-0.5" upper="3.57792194444" velocity="1.570795"/> -->
   </joint>
   <link name="arm_link_4">
@@ -208,6 +208,6 @@
     <!--<calibration rising="${arm_5_ref}" falling="${arm_5_ref}"/>-->
     <dynamics damping="1" friction="1"/>
-    <!-- <limit effort="10000.0" lower="0" upper="5.84684805556" velocity="1.570795"/> -->
-    <limit effort="10000.0" lower="-0.5" upper="5.84684805556" velocity="1.570795"/>
+    <limit effort="10000.0" lower="0" upper="5.84684805556" velocity="1.570795"/>
+    <!-- <limit effort="10000.0" lower="-0.5" upper="5.84684805556" velocity="1.570795"/> -->
   </joint>
   <link name="arm_link_5">
@@ -256,6 +256,6 @@
     <axis xyz="0 0 -1"/>
     <dynamics damping="1" friction="1"/>
-    <!-- <limit effort="10000.0" lower="0" upper="5.84684805556" velocity="1.570795"/> -->
-    <limit effort="10000.0" lower="-0.5" upper="5.84684805556" velocity="1.570795"/>
+    <limit effort="10000.0" lower="0" upper="5.84684805556" velocity="1.570795"/>
+    <!-- <limit effort="10000.0" lower="-0.5" upper="5.84684805556" velocity="1.570795"/> -->
   </joint>
   <gazebo reference="arm_link_0">

File: install/manip/share/manip/description/robot.urdf.xacro (robot description, xacro)
@@ -1 +1 @@
-/home/bfh/manip_ws/build/manip/description/robot.urdf.xacro
+/home/nbf2/manip_ws/build/manip/description/robot.urdf.xacro

File: install/manip/share/manip/description/ros2_control.xacro (robot description, xacro)
@@ -1 +1 @@
-/home/bfh/manip_ws/build/manip/description/ros2_control.xacro
+/home/nbf2/manip_ws/build/manip/description/ros2_control.xacro

File: install/manip/share/manip/description/youbot_all.xacro (robot description, xacro)
@@ -1 +1 @@
-/home/bfh/manip_ws/build/manip/description/youbot_all.xacro
+/home/nbf2/manip_ws/build/manip/description/youbot_all.xacro

File: install/manip/share/manip/description/youbot_manip.xacro (robot description, xacro)
@@ -1 +1 @@
-/home/bfh/manip_ws/build/manip/description/youbot_manip.xacro
+/home/nbf2/manip_ws/build/manip/description/youbot_manip.xacro
